File: PPMB32-E/PPMB32-E.sch (EAGLE design)
At the start: 38 parts, among them IC1 7805TV, IC2 LM3940IT-3.3, K1 ARK500/2, K2 ARK500/2, K3 ARK500/2, K4 ARK500/2, K5 ARK500/2, U1 ESP32-DEVKITC-32D

Commit message: Changed PPMB32-E scheme layout
Parts:
- removed JP4: (no value), pinhead:PINHD-1X2/90
- removed R14: (no value), rcl:R-EU_R0603
- removed U$7: MAX485DIL, MAX485:MAX485DIL
- removed U1: ESP32-DEVKITC-32D, ESP32-DEVKITC-32D:ESP32-DEVKITC-32D
- added DEVKITC: ESP32-DEVKITC-32D, ESP32-DEVKITC-32D:ESP32-DEVKITC-32D
- added K6: (no value), #PaJa_konektory:PSH02-03P
Connections:
- removed net 485_A: R14.1, U$7.A
- removed net 485_B: JP4.2, U$7.B
- removed net N$11: JP4.1, R14.2
- removed net N$14: U$7.RO
- removed net N$15: U$7.RE
- removed net N$16: U$7.DE
- removed net N$17: U$7.DI
- removed net UART2_CTS: U1.IO19
- removed net UART2_RTS: U1.IO18
- removed net UART2_RXD: U1.IO17
- removed net UART2_TXD: U1.IO16
- new net GPIO16: DEVKITC.IO16
- new net GPIO17: DEVKITC.IO17
- new net GPIO18: DEVKITC.IO18
- new net GPIO19: DEVKITC.IO19
- net +3V3: now also DEVKITC.3V3; no longer U1.3V3
- net ESP_EN: now also DEVKITC.EN; no longer U1.EN
- net EXT_5V: now also DEVKITC.EXT_5V; no longer U$7.VCC, U1.EXT_5V
- net GND: now also DEVKITC.GND1, DEVKITC.GND2, DEVKITC.GND3; no longer U$7.GND, U1.GND1, U1.GND2, U1.GND3
- net GPIO23: now also DEVKITC.IO23; no longer U1.IO23
- net GPIO26: now also DEVKITC.IO26; no longer U1.IO26
- net GPIO5: now also DEVKITC.IO5; no longer U1.IO5
- net I2C_SCL: now also DEVKITC.IO22; no longer U1.IO22
- net I2C_SDA: now also DEVKITC.IO21; no longer U1.IO21
- net INTERNAL_SENS: now also DEVKITC.IO13; no longer U1.IO13
- net N$10: now also DEVKITC.IO33; no longer U1.IO33
- net N$4: now also DEVKITC.IO34; no longer U1.IO34
- net N$8: now also DEVKITC.IO35; no longer U1.IO35
- net N$9: now also DEVKITC.IO32; no longer U1.IO32
- net ONE_WIRE: now also DEVKITC.IO15; no longer U1.IO15
- net SVN: now also DEVKITC.SENSOR_VN; no longer U1.SENSOR_VN
- net SVP: now also DEVKITC.SENSOR_VP; no longer U1.SENSOR_VP
- net UART0_RXD: now also DEVKITC.RXD0; no longer U1.RXD0
- net UART0_TXD: now also DEVKITC.TXD0; no longer U1.TXD0
- net VNH1_INA: now also DEVKITC.IO12; no longer U1.IO12
- net VNH1_INB: now also DEVKITC.IO27; no longer U1.IO27
- net VNH1_PWM: now also DEVKITC.IO14; no longer U1.IO14
- net VNH2_INA: now also DEVKITC.IO4; no longer U1.IO4
- net VNH2_INB: now also DEVKITC.IO2; no longer U1.IO2
- net VNH2_PWM: now also DEVKITC.IO0; no longer U1.IO0
- net WOVERRIDE: now also DEVKITC.IO25; no longer U1.IO25
Other:
- note added: "Connectors Sensorics"
- note added: "DevKitC"
- note added: "Power"
- note removed: "H-POWER SECTION"
